File: hardware/reflow_ctrl.sch (KiCad schematic (older format))
At the start: 18 parts, among them IC1 MAX6675, U2 MOC3063, U3 BTA41/600B, X1 Master, X2 Mains, X3 Load, X4 Thermocouple

Commit message: Add and use uMIDI.pretty generic smd packages
Parts:
- C1, C11, C2: footprint Capacitors_SMD:C_0603 -> uMIDI:Pas_0603
- C12: footprint Capacitors_SMD:C_1206 -> uMIDI:Pas_1206
- R3: footprint Resistors_SMD:R_0603 -> uMIDI:Pas_0603
- R4, R5, R6: footprint Resistors_SMD:R_1206 -> uMIDI:Pas_1206
Changed lines of the file:
@@
 F 0 "R5" V 3680 1950 50  0000 C CNN
 F 1 "360" V 3600 1950 50  0000 C CNN
-F 2 "Resistors_SMD:R_1206" V 3530 1950 30  0001 C CNN
+F 2 "uMIDI:Pas_1206" V 3530 1950 30  0001 C CNN
 F 3 "" H 3600 1950 30  0000 C CNN
 	1    3600 1950
@@
 F 0 "R6" V 5230 1200 50  0000 C CNN
 F 1 "39" V 5150 1200 50  0000 C CNN
-F 2 "Resistors_SMD:R_1206" V 5080 1200 30  0001 C CNN
+F 2 "uMIDI:Pas_1206" V 5080 1200 30  0001 C CNN
 F 3 "" H 5150 1200 30  0000 C CNN
 	1    5150 1200
@@
 F 0 "C12" H 5250 2000 50  0000 L CNN
 F 1 "10n" H 5250 1900 50  0000 L CNN
-F 2 "Capacitors_SMD:C_1206" H 5188 1700 30  0001 C CNN
+F 2 "uMIDI:Pas_1206" H 5188 1700 30  0001 C CNN
 F 3 "" H 5150 1850 60  0000 C CNN
 F 4 "630V" H 5250 1700 60  0000 L CNN "Voltage"
@@
 F 0 "R3" V 2630 1450 50  0000 C CNN
 F 1 "390" V 2550 1450 50  0000 C CNN
-F 2 "Resistors_SMD:R_0603" V 2480 1450 30  0001 C CNN
+F 2 "uMIDI:Pas_0603" V 2480 1450 30  0001 C CNN
 F 3 "" H 2550 1450 30  0000 C CNN
 	1    2550 1450
@@
 F 0 "C11" H 6050 3550 50  0000 L CNN
 F 1 "100n" H 6050 3350 50  0000 L CNN
-F 2 "Capacitors_SMD:C_0603" H 6088 3300 30  0001 C CNN
+F 2 "uMIDI:Pas_0603" H 6088 3300 30  0001 C CNN
 F 3 "" H 6050 3450 60  0001 C CNN
 	1    6050 3450
@@
 F 0 "R4" V 3680 1150 50  0000 C CNN
 F 1 "360" V 3600 1150 50  0000 C CNN
-F 2 "Resistors_SMD:R_1206" V 3530 1150 30  0001 C CNN
+F 2 "uMIDI:Pas_1206" V 3530 1150 30  0001 C CNN
 F 3 "" H 3600 1150 30  0000 C CNN
 	1    3600 1150
@@
 F 0 "C1" H 1900 4600 50  0000 L CNN
 F 1 "100n" H 1900 4400 50  0000 L CNN
-F 2 "Capacitors_SMD:C_0603" H 1938 4350 30  0001 C CNN
+F 2 "uMIDI:Pas_0603" H 1938 4350 30  0001 C CNN
 F 3 "" H 1900 4500 60  0001 C CNN
 	1    1900 4500
@@
 F 0 "C2" H 2200 4600 50  0000 L CNN
 F 1 "100n" H 2200 4400 50  0000 L CNN
-F 2 "Capacitors_SMD:C_0603" H 2238 4350 30  0001 C CNN
+F 2 "uMIDI:Pas_0603" H 2238 4350 30  0001 C CNN
 F 3 "" H 2200 4500 60  0001 C CNN
 	1    2200 4500

Commit message: Place and lock heatsink and triac
Parts:
- HS1: footprint (none) -> uMIDI:Mech-Heatsink_Fischer_SK129_STS
Changed lines of the file:
@@
 F 0 "HS1" H 4450 950 50  0000 C CNN
 F 1 "HEATSINK" H 4450 700 50  0000 C CNN
-F 2 "" H 4450 750 60  0000 C CNN
-F 3 "" H 4450 750 60  0000 C CNN
+F 2 "uMIDI:Mech-Heatsink_Fischer_SK129_STS" H 4450 750 60  0001 C CNN
+F 3 "http://www.fischerelektronik.de/web_fischer/en_GB/heatsinks/A04/Extruded%20heatsinks%20for%20PCB%20mounting/PR/SK129_50.8_/index.xhtml" H 4450 750 60  0001 C CNN
 F 4 "Fischer Elektronik" H 4450 750 60  0001 C CNN "Manufacturer"
 F 5 "SK 129-50 STS" H 4450 750 60  0001 C CNN "Manufacturer Part Number"

Commit message: Edit optotriac package; DRC clean
Parts:
- U2: footprint uMIDI:MOC3063_SMT -> uMIDI:Semi-Optotriac_MOC3063-SMD
Changed lines of the file:
@@
 F 0 "U2" H 3000 1750 50  0000 L CNN
 F 1 "MOC3063" H 3000 1350 50  0000 L CNN
-F 2 "uMIDI:MOC3063_SMT" H 3200 1550 50  0001 L CIN
+F 2 "uMIDI:Semi-Optotriac_MOC3063-SMD" H 3200 1550 50  0001 L CIN
 F 3 "https://www.fairchildsemi.com/datasheets/MO/MOC3061M.pdf" H 3175 1550 50  0001 L CNN
 F 4 "MOC3063SR2VM" H 3000 1750 50  0001 L CNN "Manufacturer Part Number"
