File: hardware/reflow_ctrl.sch (KiCad schematic (older format))
At the start: 18 parts, among them IC1 MAX6675, U2 MOC3063, U3 BTA41/600B, X1 Master, X2 Mains, X3 Load, X4 Thermocouple

Commit message: Use a smaller VDR package
Parts:
- VR1: footprint Varistors:RV_Disc_D21.5_W5.1_P10 -> Varistors:RV_Disc_D7_W4.5_P5
Changed lines of the file:
@@
 F 0 "VR1" H 5800 1650 50  0000 C TNN
 F 1 "430V" H 5800 1500 50  0000 C CNN
-F 2 "Varistors:RV_Disc_D21.5_W5.1_P10" H 5650 1550 60  0001 C CNN
+F 2 "Varistors:RV_Disc_D7_W4.5_P5" H 5650 1550 60  0001 C CNN
 F 3 "http://en.tdk.eu/inf/70/db/var_11/SIOV_Leaded_StandarD.pdf" H 5650 1550 60  0001 C CNN
 F 4 "EPCOS (TDK)" V 5710 1504 50  0001 C TNN "Manufacturer"

Commit message: Optimize header pinout and trace widths
Changed lines of the file:
@@
 Text Label 2500 3600 2    60   ~ 0
 TC_SO
-Text Label 2500 3300 2    60   ~ 0
+Text Label 1400 3200 0    60   ~ 0
 PWR
 $Comp
@@
 	1    0    0    -1
 $EndComp
-Wire Wire Line
-	3500 1450 3600 1450
-Wire Wire Line
-	3600 1450 3600 1300
-Wire Wire Line
-	3500 1650 3950 1650
-Wire Wire Line
-	3600 1650 3600 1800
-Wire Wire Line
-	3600 2100 3600 2200
-Wire Wire Line
-	3600 2200 6800 2200
-Wire Wire Line
-	5150 2000 5150 2200
-Wire Wire Line
-	5150 1700 5150 1350
-Wire Wire Line
-	3600 1000 3600 900
-Wire Wire Line
-	3600 900  5950 900
-Wire Wire Line
-	5150 1050 5150 900
-Connection ~ 5150 900
-Connection ~ 3600 1650
-Wire Wire Line
-	4450 1700 4450 2200
-Connection ~ 4450 2200
-Wire Wire Line
-	4450 1050 4450 900
-Connection ~ 4450 900
-Connection ~ 5150 2200
-Wire Wire Line
-	6150 900  6850 900
-Wire Wire Line
-	2150 1450 2400 1450
-Wire Wire Line
-	2700 1450 2900 1450
-Wire Wire Line
-	2850 1700 2850 1650
-Wire Wire Line
-	2850 1650 2900 1650
-Wire Wire Line
-	5800 3600 6050 3600
-Wire Wire Line
-	5800 3300 6050 3300
-Wire Wire Line
-	5900 3300 5900 3250
-Wire Wire Line
-	5900 3650 5900 3600
-Wire Wire Line
-	5800 3400 6800 3400
-Wire Wire Line
-	5800 3500 6800 3500
-Wire Wire Line
-	4750 3300 5100 3300
-Wire Wire Line
-	4750 3400 5100 3400
-Wire Wire Line
-	4750 3500 5100 3500
-Connection ~ 5900 3600
-Connection ~ 5900 3300
-Wire Wire Line
-	6350 1000 6850 1000
-Wire Wire Line
-	6350 1100 6850 1100
-Wire Wire Line
-	6300 2300 6800 2300
-Wire Wire Line
-	6300 2400 6800 2400
-Wire Wire Line
-	5650 1800 5650 2200
-Connection ~ 5650 2200
-Wire Wire Line
-	5650 900  5650 1300
-Connection ~ 5650 900
 Text Notes 1450 1300 0    60   ~ 0
 Nominal trigger current: 5mA (60mA max)
@@
 L +3.3V #PWR04
 U 1 1 56C0C64E
-P 2150 2950
-F 0 "#PWR04" H 2150 2800 50  0001 C CNN
-F 1 "+3.3V" H 2150 3090 50  0000 C CNN
-F 2 "" H 2150 2950 60  0000 C CNN
-F 3 "" H 2150 2950 60  0000 C CNN
-	1    2150 2950
+P 2150 3100
+F 0 "#PWR04" H 2150 2950 50  0001 C CNN
+F 1 "+3.3V" H 2150 3240 50  0000 C CNN
+F 2 "" H 2150 3100 60  0000 C CNN
+F 3 "" H 2150 3100 60  0000 C CNN
+	1    2150 3100
 	-1   0    0    -1
 $EndComp
-Wire Wire Line
-	2150 2950 2150 3200
-Wire Wire Line
-	2150 3200 2100 3200
 $Comp
 L GND #PWR05
@@
 	-1   0    0    -1
 $EndComp
-Wire Wire Line
-	1600 3600 1550 3600
-Wire Wire Line
-	1550 3600 1550 3650
 $Comp
 L C C1
@@
 	1    0    0    -1
 $EndComp
-Wire Wire Line
-	1900 4650 1900 4700
-Wire Wire Line
-	1900 4700 2200 4700
-Wire Wire Line
-	2200 4700 2200 4650
-Wire Wire Line
-	2050 4750 2050 4700
-Connection ~ 2050 4700
 $Comp
 L +3.3V #PWR07
@@
 	1    0    0    -1
 $EndComp
-Wire Wire Line
-	1900 4350 1900 4300
-Wire Wire Line
-	1900 4300 2200 4300
-Wire Wire Line
-	2200 4300 2200 4350
-Wire Wire Line
-	2050 4250 2050 4300
-Connection ~ 2050 4300
-NoConn ~ 1600 3200
 NoConn ~ 1600 3300
 NoConn ~ 1600 3400
@@
 	1    0    0    -1
 $EndComp
-Wire Wire Line
-	1000 4650 1000 4600
-Wire Wire Line
-	1000 4600 1050 4600
 $Comp
 L +3.3V #PWR011
@@
 	0    -1   -1   0
 $EndComp
-Wire Wire Line
-	1000 4400 1050 4400
 Text Label 3550 1450 0    60   ~ 0
 MOC_A1
@@
 Text Label 4950 900  0    60   ~ 0
 L_main_fused
+NoConn ~ 1600 3500
+Wire Wire Line
+	3500 1450 3600 1450
+Wire Wire Line
+	3600 1450 3600 1300
+Wire Wire Line
+	3500 1650 3950 1650
+Wire Wire Line
+	3600 1650 3600 1800
+Wire Wire Line
+	3600 2100 3600 2200
+Wire Wire Line
+	3600 2200 6800 2200
+Wire Wire Line
+	5150 2000 5150 2200
+Wire Wire Line
+	5150 1700 5150 1350
+Wire Wire Line
+	3600 1000 3600 900
+Wire Wire Line
+	3600 900  5950 900
+Wire Wire Line
+	5150 1050 5150 900
+Connection ~ 5150 900
+Connection ~ 3600 1650
+Wire Wire Line
+	4450 1700 4450 2200
+Connection ~ 4450 2200
+Wire Wire Line
+	4450 1050 4450 900
+Connection ~ 4450 900
+Connection ~ 5150 2200
+Wire Wire Line
+	6150 900  6850 900
+Wire Wire Line
+	2150 1450 2400 1450
+Wire Wire Line
+	2700 1450 2900 1450
+Wire Wire Line
+	2850 1700 2850 1650
+Wire Wire Line
+	2850 1650 2900 1650
+Wire Wire Line
+	5800 3600 6050 3600
+Wire Wire Line
+	5800 3300 6050 3300
+Wire Wire Line
+	5900 3300 5900 3250
+Wire Wire Line
+	5900 3650 5900 3600
+Wire Wire Line
+	5800 3400 6800 3400
+Wire Wire Line
+	5800 3500 6800 3500
+Wire Wire Line
+	4750 3300 5100 3300
+Wire Wire Line
+	4750 3400 5100 3400
+Wire Wire Line
+	4750 3500 5100 3500
+Connection ~ 5900 3600
+Connection ~ 5900 3300
+Wire Wire Line
+	6350 1000 6850 1000
+Wire Wire Line
+	6350 1100 6850 1100
+Wire Wire Line
+	6300 2300 6800 2300
+Wire Wire Line
+	6300 2400 6800 2400
+Wire Wire Line
+	5650 1800 5650 2200
+Connection ~ 5650 2200
+Wire Wire Line
+	5650 900  5650 1300
+Connection ~ 5650 900
+Wire Wire Line
+	2150 3100 2150 3200
+Wire Wire Line
+	2150 3200 2100 3200
+Wire Wire Line
+	1600 3600 1550 3600
+Wire Wire Line
+	1550 3600 1550 3650
+Wire Wire Line
+	1900 4650 1900 4700
+Wire Wire Line
+	1900 4700 2200 4700
+Wire Wire Line
+	2200 4700 2200 4650
+Wire Wire Line
+	2050 4750 2050 4700
+Connection ~ 2050 4700
+Wire Wire Line
+	1900 4350 1900 4300
+Wire Wire Line
+	1900 4300 2200 4300
+Wire Wire Line
+	2200 4300 2200 4350
+Wire Wire Line
+	2050 4250 2050 4300
+Connection ~ 2050 4300
+Wire Wire Line
+	1000 4650 1000 4600
+Wire Wire Line
+	1000 4600 1050 4600
+Wire Wire Line
+	1000 4400 1050 4400
 Wire Wire Line
 	2500 3400 2100 3400
@@
 	2500 3500 2100 3500
 Wire Wire Line
-	2500 3300 2100 3300
-NoConn ~ 1600 3500
+	1400 3200 1600 3200
+NoConn ~ 2100 3300
 $EndSCHEMATC

Commit message: Fix missing GND on TC-
Connections:
- wire segments 52 -> 53
Changed lines of the file:
@@
 EESchema Schematic File Version 2
-LIBS:power
-LIBS:device
-LIBS:transistors
-LIBS:conn
-LIBS:linear
-LIBS:regul
-LIBS:74xx
-LIBS:cmos4000
-LIBS:adc-dac
-LIBS:memory
-LIBS:xilinx
-LIBS:microcontrollers
-LIBS:dsp
-LIBS:microchip
-LIBS:analog_switches
-LIBS:motorola
-LIBS:texas
-LIBS:intel
-LIBS:audio
-LIBS:interface
-LIBS:digital-audio
-LIBS:philips
-LIBS:display
-LIBS:cypress
-LIBS:siliconi
-LIBS:opto
-LIBS:atmel
-LIBS:contrib
-LIBS:valves
 LIBS:reflow_ctrl-cache
 EELAYER 25 0
@@
 	1400 3200 1600 3200
 NoConn ~ 2100 3300
+$Comp
+L GND #PWR?
+U 1 1 576EC66B
+P 6650 3550
+F 0 "#PWR?" H 6650 3300 50  0001 C CNN
+F 1 "GND" H 6650 3400 50  0000 C CNN
+F 2 "" H 6650 3550 60  0000 C CNN
+F 3 "" H 6650 3550 60  0000 C CNN
+	1    6650 3550
+	1    0    0    -1
+$EndComp
+Wire Wire Line
+	6650 3550 6650 3500
+Connection ~ 6650 3500
 $EndSCHEMATC
